File: EAGLE/DazzeLiteSch.sch (EAGLE design)
At the start: 21 parts, among them U1 UPDUINO3P0, U2 74AHCT125N

Commit message: Corrected a few part numbers
Parts:
- DC1: value R-78C5.0-1.0 -> TSR_1-2450; device dc-dc-converter:R-78C5.0-1.0 -> StarLiteLib:TSR_1-2450
- S1, S3: device switch-omron:31-XX -> StarLiteLib:1-1825027-1
